File: Hardware/PCB/MKRWAN_NSK/MKRWAN_NSK.kicad_sch (KiCad schematic)
At the start: 25 parts, among them J1 Conn_01x05, J10 O2_Sensor, J13 Pont_diviseur, J2 TH_Deep_Sensor, J3 Other_Gaz_Sensor, J4 UV_IR_Sensor, J6 RGB_Sensor, J7 CO2_Sensor, J8 Pressure_Sensor, J9 TH_Surface_Sensor, U1 ARDUINO_MKR_WAN_1310

Commit message: Hardware PCB - PCB
Other:
- company: (none) -> Yulin_Vlad_Daniel_Xiaochen
- title: (none) -> Vlad_Gotupan_PCB
- moved on the sheet: NPK1
Changed lines of the file:
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@@
 	(generator_version "9.0")
 	(paper "A4")
+	(title_block
+		(title "Vlad_Gotupan_PCB")
+		(date "2025-03-08")
+		(rev "v4")
+		(company "Yulin_Vlad_Daniel_Xiaochen")
+	)
 	(junction
 		(at 243.84 153.67)
@@
 	(wire
 		(pts
-			(xy 46.99 52.07) (xy 46.99 49.53)
+			(xy 43.18 72.39) (xy 43.18 69.85)
 		)
 		(stroke
@@
 	(wire
 		(pts
-			(xy 41.91 54.61) (xy 41.91 49.53)
+			(xy 38.1 74.93) (xy 38.1 69.85)
 		)
 		(stroke
@@
 	(wire
 		(pts
-			(xy 39.37 54.61) (xy 39.37 49.53)
+			(xy 35.56 74.93) (xy 35.56 69.85)
 		)
 		(stroke
@@
 	(wire
 		(pts
-			(xy 44.45 52.07) (xy 44.45 49.53)
+			(xy 40.64 72.39) (xy 40.64 69.85)
 		)
 		(stroke
@@
 	)
 	(label "GND"
-		(at 39.37 53.34 90)
+		(at 35.56 73.66 90)
 		(effects
 			(font
@@
 	)
 	(label "5v"
-		(at 41.91 53.34 90)
+		(at 38.1 73.66 90)
 		(effects
 			(font
@@
 	)
 	(label "A_5v"
-		(at 44.45 52.07 90)
+		(at 40.64 72.39 90)
 		(effects
 			(font
@@
 	)
 	(label "B_5v"
-		(at 46.99 52.07 90)
+		(at 43.18 72.39 90)
 		(effects
 			(font
@@
 	(symbol
 		(lib_id "S4B-PH-K-S_LF__SN_:S4B-PH-K-S_LF__SN_")
-		(at 41.91 41.91 90)
+		(at 38.1 62.23 90)
 		(unit 1)
 		(exclude_from_sim no)
@@
 		(fields_autoplaced yes)
 		(property "Reference" "NPK1"
-			(at 50.8 39.3699 90)
+			(at 46.99 59.6899 90)
 			(effects
 				(font
@@
 		)
 		(property "Value" "S4B-PH-K-S_LF__SN_"
-			(at 50.8 41.9099 90)
+			(at 46.99 62.2299 90)
 			(effects
 				(font
@@
 		)
 		(property "Footprint" "Connector_JST:JST_PH_S4B-PH-K_1x04_P2.00mm_Horizontal"
-			(at 41.91 41.91 0)
+			(at 38.1 62.23 0)
 			(effects
 				(font
@@
 		)
 		(property "Datasheet" ""
-			(at 41.91 41.91 0)
+			(at 38.1 62.23 0)
 			(effects
 				(font
@@
 		)
 		(property "Description" ""
-			(at 41.91 41.91 0)
+			(at 38.1 62.23 0)
 			(effects
 				(font
@@
 		)
 		(property "MF" "JST Sales"
-			(at 41.91 41.91 0)
+			(at 38.1 62.23 0)
 			(effects
 				(font
@@
 		)
 		(property "Description_1" "Connector Header Through Hole, Right Angle 4 position 0.079 (2.00mm)"
-			(at 41.91 41.91 0)
+			(at 38.1 62.23 0)
 			(effects
 				(font
@@
 		)
 		(property "Package" "NON STANDARD-4 J.S.T."
-			(at 41.91 41.91 0)
+			(at 38.1 62.23 0)
 			(effects
 				(font
@@
 		)
 		(property "Price" "None"
-			(at 41.91 41.91 0)
+			(at 38.1 62.23 0)
 			(effects
 				(font
@@
 		)
 		(property "Check_prices" "https://www.snapeda.com/parts/S4B-PH-K-S(LF)(SN)/JST/view-part/?ref=eda"
-			(at 41.91 41.91 0)
+			(at 38.1 62.23 0)
 			(effects
 				(font
@@
 		)
 		(property "STANDARD" "Manufacturer Recommendation"
-			(at 41.91 41.91 0)
+			(at 38.1 62.23 0)
 			(effects
 				(font
@@
 		)
 		(property "SnapEDA_Link" "https://www.snapeda.com/parts/S4B-PH-K-S(LF)(SN)/JST/view-part/?ref=snap"
-			(at 41.91 41.91 0)
+			(at 38.1 62.23 0)
 			(effects
 				(font
@@
 		)
 		(property "MP" "S4B-PH-K-S(LF)(SN)"
-			(at 41.91 41.91 0)
+			(at 38.1 62.23 0)
 			(effects
 				(font
@@
 		)
 		(property "Availability" "In Stock"
-			(at 41.91 41.91 0)
+			(at 38.1 62.23 0)
 			(effects
 				(font
@@
 		)
 		(property "MANUFACTURER" "JST"
-			(at 41.91 41.91 0)
+			(at 38.1 62.23 0)
 			(effects
 				(font
